Commit message: bblaze updates

File: moveo_urdf/urdf/moveo_urdf_new.urdf (robot description, URDF)
Before this commit: robot moveo_urdf_5, 12 links, 11 joints
Links:
- added link Link_6, mass 0.19875; collision mesh filename=package://moveo_urdf_5/meshes/Link_6.STL; visual mesh filename=package://moveo_urdf_5/meshes/Link_6.STL
Joints:
- added joint Joint_6: type revolute, parent Link_5, child Link_6, origin xyz=-0.0021346 0.053041 0.0016936 rpy=-1.5639 -0.091135 -0.00062919, axis 0 1 0, limit lower=-1 upper=1 effort=5 velocity=1
- joint Gripper_Idol_Gear_Joint: parent Link_5 -> Link_6
